Commit message: simulation model correctly loaded to gazebo

File: ros2_ws/src/turtlebot3_description/urdf/turtlebot3_waffle.urdf (robot description, URDF)
Before this commit: robot turtlebot3_waffle, 13 links, 12 joints
Links:
- removed link ${namespace}imu_link
Joints:
- removed joint ${namespace}imu_joint
