Commit message: fix: correct wrong CoM and add joint_state_publisher in launch file

File: ros2_ws/src/do_description/urdf/do/do_trailer.xacro (robot description, xacro)
@@ -16,5 +16,5 @@
         </collision>
         <xacro:box_inertia m="${total_mass * 0.8 * 0.3}" l="${trailer_length}" w="${trailer_width}" h="${trailer_height}"
-                       xyz="0 0 ${trailer_height / 2.0 + trailer_ground_clearance}"  rpy="0 0 0"/>
+                       xyz="-${trailer_visual_x_offset} 0 0"  rpy="0 0 0"/>
     </link>
     <link name="right_caster_wheel">
@@ -50,9 +50,10 @@
         <xacro:sphere_inertia m="${total_mass * 0.5 * 0.5 * 0.1}" r="${caster_wheels_radius}" xyz="0 0 0" rpy="0 0 0"/>
     </link>
-    <joint name="trailer_joint" type="continuous">
+    <joint name="trailer_joint" type="revolute">
 	    <parent link="base_link"/>
 	    <child link="trailer"/>
 	    <origin xyz="-${trailer_axis_x_offset} 0 ${trailer_axis_height}" rpy="0 0 0"/>
 	    <axis xyz="0 1 0"/>
+        <limit effort="10" velocity="1.0" lower="-0.6" upper="0.6" />
 	</joint>
 	<joint name="right_caster_wheel_joint" type="fixed">
