Commit message: visually correct model (incorrect inertia)

File: ros2_ws/src/do_description/urdf/do/do.urdf.xacro (robot description, xacro)
@@ -1,20 +1,32 @@
 <?xml version="1.0"?>
 <robot name="do" xmlns:xacro="http://wwww.ros.org/wiki/xacro">
-	<xacro:property name="cm_to_m" value="0.01"/>
-	<xacro:property name="base_link_length" value="${9.1 * cm_to_m}"/>
-	<xacro:property name="base_link_width" value="${11.2 * cm_to_m}"/>
-	<xacro:property name="base_link_height" value="${4.4 * cm_to_m}"/>
-	<xacro:property name="base_link_ground_clearance" value="${0.45 * cm_to_m}"/>
-	<xacro:property name="ball_wheel_radius" value="${0.9 * cm_to_m}"/>
-	<xacro:property name="ball_wheel_x_offset" value="${3.5 * cm_to_m}"/>
-	<xacro:property name="wheels_radius" value="${2.2 * cm_to_m}"/>
-	<xacro:property name="wheels_length" value="${1.5 * cm_to_m}"/>
-	<xacro:property name="wheels_x_offset" value="${2.5 * cm_to_m}"/>
-	<xacro:property name="wheels_spacing" value="${9.35 * cm_to_m}"/>
+	<xacro:property name="mm_to_m" value="0.001"/>
+	<xacro:property name="base_link_length" value="${204 * mm_to_m}"/>
+	<xacro:property name="base_link_width" value="${460 * mm_to_m}"/>
+	<xacro:property name="base_link_height" value="${156 * mm_to_m}"/>
+	<xacro:property name="base_link_ground_clearance" value="${20.5 * mm_to_m}"/>
+	<xacro:property name="ball_wheels_radius" value="${9.5 * mm_to_m}"/>
+	<xacro:property name="ball_wheels_x_offset" value="${79.3 * mm_to_m}"/>
+	<xacro:property name="ball_wheels_spacing" value="${413.5 * mm_to_m}"/>
+	<xacro:property name="wheels_radius" value="${55.5 * mm_to_m}"/>
+	<xacro:property name="wheels_width" value="${44 * mm_to_m}"/>
+	<xacro:property name="wheels_x_offset" value="${40 * mm_to_m}"/>
+	<xacro:property name="wheels_spacing" value="${414.7 * mm_to_m}"/>
+	<xacro:property name="trailer_length" value="${180 * mm_to_m}"/>
+	<xacro:property name="trailer_width" value="${265 * mm_to_m}"/>
+	<xacro:property name="trailer_height" value="${156 * mm_to_m}"/>
+	<xacro:property name="trailer_ground_clearance" value="${20.5 * mm_to_m}"/>
+	<xacro:property name="trailer_visual_x_offset" value="${158 * mm_to_m}"/>
+	<xacro:property name="trailer_axis_x_offset" value="${78 * mm_to_m}"/>
+	<xacro:property name="trailer_axis_height" value="${100.5 * mm_to_m}"/>
+	<xacro:property name="castor_wheels_radius" value="${16 * mm_to_m}"/>
+	<xacro:property name="castor_wheels_x_offset" value="${215 * mm_to_m}"/>
+	<xacro:property name="castor_wheels_spacing" value="${331.2 * mm_to_m}"/>
 	<xacro:property name="total_mass" value="0.27"/>
 	<xacro:include filename="materials.xacro"/>
 	<xacro:include filename="do_inertia.xacro"/>
 	<xacro:include filename="do_chassis.xacro"/>
+	<xacro:include filename="do_trailer.xacro"/>
 	<xacro:include filename="gazebo.xacro"/>
-	<xacro:include filename="proximity_sensors.xacro"/>
+	<!-- <xacro:include filename="proximity_sensors.xacro"/> -->
 </robot>

File: ros2_ws/src/do_description/urdf/do/do_chassis.xacro (robot description, xacro)
@@ -22,5 +22,5 @@
             <origin xyz="0 0 0" rpy="${pi / 2.0} 0 0"/>
             <geometry>
-                <cylinder length="${wheels_length}" radius="${wheels_radius}"/>
+                <cylinder length="${wheels_width}" radius="${wheels_radius}"/>
             </geometry>
             <material name="black"/>
@@ -29,8 +29,8 @@
             <origin xyz="0 0 0" rpy="${pi / 2.0} 0 0"/>
             <geometry>
-                <cylinder length="${wheels_length}" radius="${wheels_radius}"/>
+                <cylinder length="${wheels_width}" radius="${wheels_radius}"/>
             </geometry>
         </collision>
-        <xacro:cylinder_inertia m="${total_mass * 0.2 * 0.5}" r="${wheels_radius}" h="${wheels_length}"
+        <xacro:cylinder_inertia m="${total_mass * 0.2 * 0.5}" r="${wheels_radius}" h="${wheels_width}"
                             xyz="0 0 0" rpy="${pi / 2.0} 0 0"/>
     </link>
@@ -39,5 +39,5 @@
             <origin xyz="0 0 0" rpy="${pi / 2.0} 0 0"/>
             <geometry>
-                <cylinder length="${wheels_length}" radius="${wheels_radius}"/>
+                <cylinder length="${wheels_width}" radius="${wheels_radius}"/>
             </geometry>
             <material name="black"/>
@@ -46,15 +46,15 @@
             <origin xyz="0 0 0" rpy="${pi / 2.0} 0 0"/>
             <geometry>
-                <cylinder length="${wheels_length}" radius="${wheels_radius}"/>
+                <cylinder length="${wheels_width}" radius="${wheels_radius}"/>
             </geometry>
         </collision>
-        <xacro:cylinder_inertia m="${total_mass * 0.2 * 0.5}" r="${wheels_radius}" h="${wheels_length}"
+        <xacro:cylinder_inertia m="${total_mass * 0.2 * 0.5}" r="${wheels_radius}" h="${wheels_width}"
                             xyz="0 0 0" rpy="${pi / 2.0} 0 0"/>
     </link>
-    <link name="ball_wheel">
+    <link name="right_ball_wheel">
         <visual>
             <origin xyz="0 0 0" rpy="0 0 0"/>
             <geometry>
-                <sphere radius="${ball_wheel_radius}"/>
+                <sphere radius="${ball_wheels_radius}"/>
             </geometry>
             <material name="white"/>
@@ -63,8 +63,24 @@
             <origin xyz="0 0 0" rpy="0 0 0"/>
             <geometry>
-                <sphere radius="${ball_wheel_radius}"/>
+                <sphere radius="${ball_wheels_radius}"/>
             </geometry>
         </collision>
-        <xacro:sphere_inertia m="${total_mass * 0.8 * 0.05}" r="${ball_wheel_radius}" xyz="0 0 0" rpy="0 0 0"/>
+        <xacro:sphere_inertia m="${total_mass * 0.8 * 0.05}" r="${ball_wheels_radius}" xyz="0 0 0" rpy="0 0 0"/>
+    </link>
+    <link name="left_ball_wheel">
+        <visual>
+            <origin xyz="0 0 0" rpy="0 0 0"/>
+            <geometry>
+                <sphere radius="${ball_wheels_radius}"/>
+            </geometry>
+            <material name="white"/>
+        </visual>
+        <collision>
+            <origin xyz="0 0 0" rpy="0 0 0"/>
+            <geometry>
+                <sphere radius="${ball_wheels_radius}"/>
+            </geometry>
+        </collision>
+        <xacro:sphere_inertia m="${total_mass * 0.8 * 0.05}" r="${ball_wheels_radius}" xyz="0 0 0" rpy="0 0 0"/>
     </link>
     <joint name="right_wheel_joint" type="continuous">
@@ -82,8 +98,13 @@
         <dynamics damping="0.1" friction="0.2"/>
 	</joint>
-	<joint name="ball_wheel_joint" type="fixed">
+	<joint name="right_ball_wheel_joint" type="fixed">
 	    <parent link="base_link"/>
-	    <child link="ball_wheel"/>
-	    <origin xyz="${ball_wheel_x_offset} 0 ${ball_wheel_radius}" rpy="0 0 0"/>
+	    <child link="right_ball_wheel"/>
+	    <origin xyz="${ball_wheels_x_offset} -${ball_wheels_spacing / 2.0} ${ball_wheels_radius}" rpy="0 0 0"/>
 	</joint>
+    <joint name="left_ball_wheel_joint" type="fixed">
+        <parent link="base_link"/>
+        <child link="left_ball_wheel"/>
+        <origin xyz="${ball_wheels_x_offset} ${ball_wheels_spacing / 2.0} ${ball_wheels_radius}" rpy="0 0 0"/>
+    </joint>
 </robot>

Commit message: Simple vel control from practicals working

File: ros2_ws/src/do_description/urdf/do/do.urdf.xacro (robot description, xacro)
@@ -20,7 +20,7 @@
 	<xacro:property name="trailer_axis_x_offset" value="${78 * mm_to_m}"/>
 	<xacro:property name="trailer_axis_height" value="${100.5 * mm_to_m}"/>
-	<xacro:property name="castor_wheels_radius" value="${16 * mm_to_m}"/>
-	<xacro:property name="castor_wheels_x_offset" value="${215 * mm_to_m}"/>
-	<xacro:property name="castor_wheels_spacing" value="${331.2 * mm_to_m}"/>
+	<xacro:property name="caster_wheels_radius" value="${16 * mm_to_m}"/>
+	<xacro:property name="caster_wheels_x_offset" value="${215 * mm_to_m}"/>
+	<xacro:property name="caster_wheels_spacing" value="${331.2 * mm_to_m}"/>
 	<xacro:property name="total_mass" value="0.27"/>
 	<xacro:include filename="materials.xacro"/>

File: ros2_ws/src/do_description/urdf/do/do_trailer.xacro (robot description, xacro)
@@ -18,9 +18,9 @@
                        xyz="0 0 ${trailer_height / 2.0 + trailer_ground_clearance}"  rpy="0 0 0"/>
     </link>
-    <link name="right_castor_wheel">
+    <link name="right_caster_wheel">
         <visual>
             <origin xyz="0 0 0" rpy="0 0 0"/>
             <geometry>
-                <sphere radius="${castor_wheels_radius}"/>
+                <sphere radius="${caster_wheels_radius}"/>
             </geometry>
             <material name="white"/>
@@ -29,14 +29,14 @@
             <origin xyz="0 0 0" rpy="0 0 0"/>
             <geometry>
-                <sphere radius="${castor_wheels_radius}"/>
+                <sphere radius="${caster_wheels_radius}"/>
             </geometry>
         </collision>
-        <xacro:sphere_inertia m="${total_mass * 0.8 * 0.05}" r="${castor_wheels_radius}" xyz="0 0 0" rpy="0 0 0"/>
+        <xacro:sphere_inertia m="${total_mass * 0.8 * 0.05}" r="${caster_wheels_radius}" xyz="0 0 0" rpy="0 0 0"/>
     </link>
-    <link name="left_castor_wheel">
+    <link name="left_caster_wheel">
         <visual>
             <origin xyz="0 0 0" rpy="0 0 0"/>
             <geometry>
-                <sphere radius="${castor_wheels_radius}"/>
+                <sphere radius="${caster_wheels_radius}"/>
             </geometry>
             <material name="white"/>
@@ -45,8 +45,8 @@
             <origin xyz="0 0 0" rpy="0 0 0"/>
             <geometry>
-                <sphere radius="${castor_wheels_radius}"/>
+                <sphere radius="${caster_wheels_radius}"/>
             </geometry>
         </collision>
-        <xacro:sphere_inertia m="${total_mass * 0.8 * 0.05}" r="${castor_wheels_radius}" xyz="0 0 0" rpy="0 0 0"/>
+        <xacro:sphere_inertia m="${total_mass * 0.8 * 0.05}" r="${caster_wheels_radius}" xyz="0 0 0" rpy="0 0 0"/>
     </link>
     <joint name="trailer_joint" type="continuous">
@@ -56,13 +56,13 @@
 	    <axis xyz="0 1 0"/>
 	</joint>
-	<joint name="right_castor_wheel_joint" type="fixed">
+	<joint name="right_caster_wheel_joint" type="fixed">
 	    <parent link="trailer"/>
-	    <child link="right_castor_wheel"/>
-	    <origin xyz="-${castor_wheels_x_offset} -${castor_wheels_spacing / 2.0} ${castor_wheels_radius - (trailer_height / 2.0 + trailer_ground_clearance)}" rpy="0 0 0"/>
+	    <child link="right_caster_wheel"/>
+	    <origin xyz="-${caster_wheels_x_offset} -${caster_wheels_spacing / 2.0} ${caster_wheels_radius - (trailer_height / 2.0 + trailer_ground_clearance)}" rpy="0 0 0"/>
 	</joint>
-    <joint name="left_castor_wheel_joint" type="fixed">
+    <joint name="left_caster_wheel_joint" type="fixed">
         <parent link="trailer"/>
-        <child link="left_castor_wheel"/>
-        <origin xyz="-${castor_wheels_x_offset} ${castor_wheels_spacing / 2.0} ${castor_wheels_radius - (trailer_height / 2.0 + trailer_ground_clearance)}" rpy="0 0 0"/>
+        <child link="left_caster_wheel"/>
+        <origin xyz="-${caster_wheels_x_offset} ${caster_wheels_spacing / 2.0} ${caster_wheels_radius - (trailer_height / 2.0 + trailer_ground_clearance)}" rpy="0 0 0"/>
     </joint>
 </robot>

File: ros2_ws/src/do_description/urdf/do/gazebo.xacro (robot description, xacro)
@@ -1,10 +1,19 @@
 <?xml version="1.0"?>
 <robot xmlns:xacro="http://wwww.ros.org/wiki/xacro">
-    <gazebo reference="caster_wheel_link">
+    <gazebo reference="right_ball_wheel">
         <mu1 value="0.31" />
         <mu2 value="0.31" />
     </gazebo>
-    <gazebo reference="base_link">
-        <material>Gazebo/White</material>
+    <gazebo reference="left_ball_wheel">
+        <mu1 value="0.31" />
+        <mu2 value="0.31" />
+    </gazebo>
+    <gazebo reference="right_caster_wheel">
+        <mu1 value="0.31" />
+        <mu2 value="0.31" />
+    </gazebo>
+    <gazebo reference="left_caster_wheel">
+        <mu1 value="0.31" />
+        <mu2 value="0.31" />
     </gazebo>
     <gazebo reference="right_wheel">
@@ -13,7 +22,4 @@
     <gazebo reference="left_wheel">
         <material>Gazebo/Black</material>
-    </gazebo>
-    <gazebo reference="ball_wheel">
-        <material>Gazebo/White</material>
     </gazebo>
     <gazebo>

Commit message: teleop simulation with keyboard working

File: ros2_ws/src/do_description/urdf/do/do.urdf.xacro (robot description, xacro)
@@ -25,9 +25,10 @@
 	<xacro:property name="caster_wheels_x_offset" value="${215 * mm_to_m}"/>
 	<xacro:property name="caster_wheels_spacing" value="${331.2 * mm_to_m}"/>
-	<xacro:property name="total_mass" value="0.27"/>
+	<xacro:property name="total_mass" value="5.0"/>
 	<xacro:include filename="materials.xacro"/>
 	<xacro:include filename="do_inertia.xacro"/>
 	<xacro:include filename="do_chassis.xacro"/>
 	<xacro:include filename="do_trailer.xacro"/>
+	<xacro:include filename="gazebo.xacro"/>
 	<!-- <xacro:include filename="proximity_sensors.xacro"/> -->
 	<!-- Use ros2_control by default, otherwise go back to legacy -->
@@ -36,5 +37,5 @@
     </xacro:if>
     <xacro:unless value="$(arg use_ros2_control)">
-        <xacro:include filename="gazebo.xacro" />
+        <xacro:include filename="gazeb_diff_control.xacro" />
     </xacro:unless>
 </robot>

File: ros2_ws/src/do_description/urdf/do/do_trailer.xacro (robot description, xacro)
@@ -54,5 +54,5 @@
 	    <child link="trailer"/>
 	    <origin xyz="-${trailer_axis_x_offset} 0 ${trailer_axis_height}" rpy="0 0 0"/>
-	    <axis xyz="0 1 0"/>
+	    <axis xyz="0 0 1"/>
 	</joint>
 	<joint name="right_caster_wheel_joint" type="fixed">

File: ros2_ws/src/do_description/urdf/do/gazebo.xacro (robot description, xacro)
@@ -23,24 +23,3 @@
         <material>Gazebo/Black</material>
     </gazebo>
-    <gazebo>
-        <plugin name="diff_drive_controller" filename="libgazebo_ros_diff_drive.so">
-        <!-- Update rate in Hz -->
-        <update_rate>50</update_rate>
-        <!-- wheels -->
-        <left_joint>left_wheel_joint</left_joint>
-        <right_joint>right_wheel_joint</right_joint>
-        <!-- kinematics -->
-        <wheel_separation>${wheels_spacing}</wheel_separation>
-        <wheel_diameter>${wheels_radius * 2.0}</wheel_diameter>
-        <!-- input -->
-        <command_topic>cmd_vel</command_topic>
-        <!-- output -->
-        <publish_odom>true</publish_odom>
-        <publish_odom_tf>true</publish_odom_tf>
-        <publish_wheel_tf>true</publish_wheel_tf>
-        <odometry_topic>odom</odometry_topic>
-        <odometry_frame>odom</odometry_frame>
-        <robot_base_frame>base_link</robot_base_frame>
-        </plugin>
-    </gazebo>
 </robot>

Commit message: fix bugs in simu and update  masses

File: ros2_ws/src/do_description/urdf/do/do.urdf.xacro (robot description, xacro)
@@ -25,18 +25,10 @@
 	<xacro:property name="caster_wheels_x_offset" value="${215 * mm_to_m}"/>
 	<xacro:property name="caster_wheels_spacing" value="${331.2 * mm_to_m}"/>
-	<xacro:property name="total_mass" value="5.0"/>
+	<xacro:property name="total_mass" value="3.1"/>
 	<xacro:include filename="materials.xacro"/>
 	<xacro:include filename="do_inertia.xacro"/>
 	<xacro:include filename="do_chassis.xacro"/>
 	<xacro:include filename="do_trailer.xacro"/>
+	<xacro:include filename="lidar.xacro"/>
 	<xacro:include filename="gazebo.xacro"/>
-	<!-- <xacro:include filename="proximity_sensors.xacro"/> -->
-	<xacro:include filename="lidar.xacro"/>
-	<!-- Use ros2_control by default, otherwise go back to legacy -->
-	<xacro:if value="$(arg use_ros2_control)">
-        <xacro:include filename="ros2_control.xacro" />
-    </xacro:if>
-    <xacro:unless value="$(arg use_ros2_control)">
-        <xacro:include filename="gazeb_diff_control.xacro" />
-    </xacro:unless>
 </robot>

File: ros2_ws/src/do_description/urdf/do/do_chassis.xacro (robot description, xacro)
@@ -15,5 +15,5 @@
             </geometry>
         </collision>
-        <xacro:box_inertia m="${total_mass * 0.8 * 0.95}" l="${base_link_length}" w="${base_link_width}" h="${base_link_height}"
+        <xacro:box_inertia m="${total_mass * 0.7 * 0.66}" l="${base_link_length}" w="${base_link_width}" h="${base_link_height}"
                        xyz="0 0 ${base_link_height / 2.0 + base_link_ground_clearance}"  rpy="0 0 0"/>
     </link>
@@ -66,5 +66,5 @@
             </geometry>
         </collision>
-        <xacro:sphere_inertia m="${total_mass * 0.8 * 0.05}" r="${ball_wheels_radius}" xyz="0 0 0" rpy="0 0 0"/>
+        <xacro:sphere_inertia m="${total_mass * 0.5 * 0.5 * 0.1}" r="${ball_wheels_radius}" xyz="0 0 0" rpy="0 0 0"/>
     </link>
     <link name="left_ball_wheel">
@@ -82,5 +82,5 @@
             </geometry>
         </collision>
-        <xacro:sphere_inertia m="${total_mass * 0.8 * 0.05}" r="${ball_wheels_radius}" xyz="0 0 0" rpy="0 0 0"/>
+        <xacro:sphere_inertia m="${total_mass * 0.5 * 0.5 * 0.1}" r="${ball_wheels_radius}" xyz="0 0 0" rpy="0 0 0"/>
     </link>
     <joint name="right_wheel_joint" type="continuous">

File: ros2_ws/src/do_description/urdf/do/do_trailer.xacro (robot description, xacro)
@@ -15,5 +15,5 @@
             </geometry>
         </collision>
-        <xacro:box_inertia m="${total_mass * 0.8 * 0.95}" l="${trailer_length}" w="${trailer_width}" h="${trailer_height}"
+        <xacro:box_inertia m="${total_mass * 0.7 * 0.34}" l="${trailer_length}" w="${trailer_width}" h="${trailer_height}"
                        xyz="0 0 ${trailer_height / 2.0 + trailer_ground_clearance}"  rpy="0 0 0"/>
     </link>
@@ -32,5 +32,5 @@
             </geometry>
         </collision>
-        <xacro:sphere_inertia m="${total_mass * 0.8 * 0.05}" r="${caster_wheels_radius}" xyz="0 0 0" rpy="0 0 0"/>
+        <xacro:sphere_inertia m="${total_mass * 0.5 * 0.5 * 0.1}" r="${caster_wheels_radius}" xyz="0 0 0" rpy="0 0 0"/>
     </link>
     <link name="left_caster_wheel">
@@ -48,5 +48,5 @@
             </geometry>
         </collision>
-        <xacro:sphere_inertia m="${total_mass * 0.8 * 0.05}" r="${caster_wheels_radius}" xyz="0 0 0" rpy="0 0 0"/>
+        <xacro:sphere_inertia m="${total_mass * 0.5 * 0.5 * 0.1}" r="${caster_wheels_radius}" xyz="0 0 0" rpy="0 0 0"/>
     </link>
     <joint name="trailer_joint" type="continuous">
@@ -54,5 +54,5 @@
 	    <child link="trailer"/>
 	    <origin xyz="-${trailer_axis_x_offset} 0 ${trailer_axis_height}" rpy="0 0 0"/>
-	    <axis xyz="0 0 1"/>
+	    <axis xyz="0 1 0"/>
 	</joint>
 	<joint name="right_caster_wheel_joint" type="fixed">

File: ros2_ws/src/do_description/urdf/do/gazebo.xacro (robot description, xacro)
@@ -23,3 +23,10 @@
         <material>Gazebo/Black</material>
     </gazebo>
+    <!-- Use ros2_control by default, otherwise go back to legacy -->
+    <xacro:if value="$(arg use_ros2_control)">
+        <xacro:include filename="gazebo_ros2_control.xacro" />
+    </xacro:if>
+    <xacro:unless value="$(arg use_ros2_control)">
+        <xacro:include filename="gazebo_diff_control.xacro" />
+    </xacro:unless>
 </robot>

Commit message: correct lidar position and orientation

File: ros2_ws/src/do_description/urdf/do/do.urdf.xacro (robot description, xacro)
@@ -25,4 +25,9 @@
 	<xacro:property name="caster_wheels_x_offset" value="${215 * mm_to_m}"/>
 	<xacro:property name="caster_wheels_spacing" value="${331.2 * mm_to_m}"/>
+	<xacro:property name="lidar_radius" value="${35 * mm_to_m}"/>
+	<xacro:property name="lidar_height" value="${20 * mm_to_m}"/>
+	<xacro:property name="lidar_x_offset" value="${85 * mm_to_m}"/>
+	<xacro:property name="lidar_z_offset" value="${252 * mm_to_m}"/>
+	<xacro:property name="lidar_mass" value="${0.170}"/>
 	<xacro:property name="total_mass" value="3.1"/>
 	<xacro:include filename="materials.xacro"/>
@@ -30,5 +35,5 @@
 	<xacro:include filename="do_chassis.xacro"/>
 	<xacro:include filename="do_trailer.xacro"/>
-	<!-- <xacro:include filename="lidar.xacro"/> -->
+	<xacro:include filename="lidar.xacro"/>
 	<xacro:include filename="gazebo.xacro"/>
 </robot>

File: ros2_ws/src/do_description/urdf/do/lidar.xacro (robot description, xacro)
@@ -1,30 +1,28 @@
 <?xml version="1.0"?>
 <robot name="do" xmlns:xacro="http://www.ros.org/wiki/xacro">
-    <link name="lidar_link">
-    <inertial>
-        <origin xyz="0 0 0" rpy="0 0 0"/>
-        <mass value="0.125"/>
-        <inertia ixx="0.001"  ixy="0"  ixz="0" iyy="0.001" iyz="0" izz="0.001" />
-    </inertial>
-    <collision>
-        <origin xyz="0 0 0" rpy="0 0 0"/>
-        <geometry>
-        <cylinder radius="0.0508" length="0.055"/>
-        </geometry>
-    </collision>
-    <visual>
-        <origin xyz="0 0 0" rpy="0 0 0"/>
-        <geometry>
-        <cylinder radius="0.0508" length="0.055"/>
-        </geometry>
-    </visual>
+    <link name="laser">
+        <visual>
+            <origin xyz="0 0 0" rpy="0 0 0"/>
+            <geometry>
+                <cylinder radius="${lidar_radius}" length="${lidar_height}"/>
+            </geometry>
+            <material name="black"/>
+        </visual>
+        <collision>
+            <origin xyz="0 0 0" rpy="0 0 0"/>
+            <geometry>
+                <cylinder radius="${lidar_radius}" length="${lidar_height}"/>
+            </geometry>
+        </collision>
+        <xacro:cylinder_inertia m="${lidar_mass}" r="${lidar_radius}" h="${lidar_height}"
+                            xyz="0 0 0" rpy="0 0 0"/>
     </link>
-    <joint name="lidar_joint" type="fixed">
+    <joint name="laser_joint" type="fixed">
         <parent link="base_link"/>
-        <child link="lidar_link"/>
-        <origin xyz="0 0 0.20" rpy="0 0 0"/>
+        <child link="laser"/>
+        <origin xyz="${lidar_x_offset} 0 ${lidar_z_offset}" rpy="0 0 -${pi / 2.0}"/>
     </joint>
-    <gazebo reference="lidar_link">
-        <sensor name="lidar" type="ray">
+    <gazebo reference="laser">
+        <sensor name="laser" type="ray">
             <always_on>true</always_on>
             <visualize>true</visualize>
@@ -55,5 +53,5 @@
             </ros>
             <output_type>sensor_msgs/LaserScan</output_type>
-            <frame_name>lidar_link</frame_name>
+            <frame_name>laser</frame_name>
             </plugin>
         </sensor>
