Commit message: correct missing lines for do compatibility

File: ros2_ws/src/do_description/urdf/do/gazebo_ros2_control.xacro (robot description, xacro)
@@ -41,4 +41,8 @@
             <state_interface name="velocity"/>
         </joint>
+        <joint name="duplo_counter">
+            <command_interface name="position"/>
+            <state_interface name="position"/>
+        </joint>
     </ros2_control>
 </robot>
