Commit message: add draft of logic bug needs debugging

File: ros2_ws/src/da_description/urdf/da/ros2_control.xacro (robot description, xacro)
@@ -34,4 +34,8 @@
             <state_interface name="velocity"/>
         </joint>
+        <joint name="robot_mode">
+            <command_interface name="position"/>
+            <state_interface name="position"/>
+        </joint>
     </ros2_control>
 </robot>
