Commit message: sweeper node is running but brushes are not turning

File: ros2_ws/src/da_description/urdf/da/gazebo_ros2_control.xacro (robot description, xacro)
@@ -41,4 +41,8 @@
             <state_interface name="velocity"/>
         </joint>
+        <joint name="sweeper_mode">
+            <command_interface name="position"/>
+            <state_interface name="position"/>
+        </joint>
     </ros2_control>
 </robot>

Commit message: add duplo_count to the ros2_control interface (check /joint_states topic to access it)

File: ros2_ws/src/da_description/urdf/da/gazebo_ros2_control.xacro (robot description, xacro)
@@ -45,4 +45,8 @@
             <state_interface name="position"/>
         </joint>
+        <joint name="duplo_counter">
+            <command_interface name="position"/>
+            <state_interface name="position"/>
+        </joint>
     </ros2_control>
 </robot>
